File: Battery.kicad_sch (KiCad schematic)
At the start: 5 parts, among them J1 USB_A

Commit message: up
Parts:
- added J?: Conn_01x06_Female, Connector_TE-Connectivity:TE_826576-6_1x06_P3.96mm_Vertical, symbol Connector:Conn_01x06_Female
Changed lines of the file:
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@@
     (pin "2")
+  )
+  (symbol (lib_id "Connector:Conn_01x06_Female") (at 67.31 81.28 0) (unit 1)
+    (in_bom yes) (on_board yes) (fields_autoplaced)
+    (property "Reference" "J?" (id 0) (at 68.58 81.2799 0)
+      (effects (font (size 1.27 1.27)) (justify left))
+    )
+    (property "Value" "Conn_01x06_Female" (id 1) (at 68.58 83.8199 0)
+      (effects (font (size 1.27 1.27)) (justify left))
+    )
+    (property "Footprint" "Connector_TE-Connectivity:TE_826576-6_1x06_P3.96mm_Vertical" (id 2) (at 67.31 81.28 0)
+      (effects (font (size 1.27 1.27)) hide)
+    )
+    (property "Datasheet" "~" (id 3) (at 67.31 81.28 0)
+      (effects (font (size 1.27 1.27)) hide)
+    )
+    (pin "1")
+    (pin "2")
+    (pin "3")
+    (pin "4")
+    (pin "5")
+    (pin "6")
   )
   (symbol (lib_id "power:GND") (at 96.52 97.79 0) (unit 1)
@@
       (reference "J1") (unit 1) (value "USB_A") (footprint "Connector_USB:USB_A_Molex_67643_Horizontal")
     )
+    (path "/ef8c9c2e-fdc4-4c3d-8606-0f75099b4372"
+      (reference "J?") (unit 1) (value "Conn_01x06_Female") (footprint "Connector_TE-Connectivity:TE_826576-6_1x06_P3.96mm_Vertical")
+    )
     (path "/d9352029-c9e7-4c14-8e73-445fcae555b0"
